Commit message: [update] set correct limit in urdf

File: robots/sia20f.urdf (robot description, URDF)
Before this commit: robot sia20f, 8 links, 7 joints
Joints:
- joint joint_b: limit lower=-1.9198 upper=1.9198 effort=100 velocity=3.4 -> lower=-1.9198 upper=1.9198 effort=100 velocity=3.4906
- joint joint_e: limit lower=-2.9670 upper=2.9670 effort=100 velocity=3.1415 -> lower=-2.9670 upper=2.9670 effort=100 velocity=2.9670
- joint joint_l: limit lower=-1.9198 upper=1.19198 effort=100 velocity=3.1415 -> lower=-1.9198 upper=1.9198 effort=100 velocity=2.2689
- joint joint_r: limit lower=-3.1415 upper=3.1414 effort=100 velocity=3.1415 -> lower=-3.1415 upper=3.1414 effort=100 velocity=3.4906
- joint joint_s: limit lower=-3.1415 upper=3.1415 effort=100 velocity=3.1415 -> lower=-3.1415 upper=3.1415 effort=100 velocity=2.2689
- joint joint_u: limit lower=-2.9670 upper=2.9670 effort=100 velocity=3.1415 -> lower=-2.9670 upper=2.9670 effort=100 velocity=2.9670
