Commit message: [update] start gazebo

File: robots/sia20.urdf.xacro (robot description, xacro)
@@ -19,32 +19,34 @@
 		<origin xyz="0 0 0" rpy="0 0 0" />
 	</xacro:macro>
-	<xacro:macro name="origin_base_link">
+	<xacro:macro name="inertia_origin_base_link">
 		<origin xyz="-0.05327 0.066798 0.00014271" rpy="0 0 0" />
 	</xacro:macro>
-	<xacro:macro name="origin_link_s">
+	<xacro:macro name="inertia_origin_link_s">
         <origin xyz="7.8023E-07 0.18911 -0.015611" rpy="0 0 0" />
 	</xacro:macro>
-	<xacro:macro name="origin_link_l">
+	<xacro:macro name="inertia_origin_link_l">
         <origin xyz="1.6057E-05 0.10201 0.041335" rpy="0 0 0" />
 	</xacro:macro>
-	<xacro:macro name="origin_link_e">
+	<xacro:macro name="inertia_origin_link_e">
         <origin xyz="3.9186E-05 0.16471 0.020774" rpy="0 0 0" />
 	</xacro:macro>
-	<xacro:macro name="origin_link_u">
+	<xacro:macro name="inertia_origin_link_u">
         <origin xyz="-7.9992E-07 0.08472 -0.032542" rpy="0 0 0" />
 	</xacro:macro>
-	<xacro:macro name="origin_link_r">
+	<xacro:macro name="inertia_origin_link_r">
         <origin xyz="4.8678E-06 0.12569 -0.02028" rpy="0 0 0" />
 	</xacro:macro>
-	<xacro:macro name="origin_link_b">
+	<xacro:macro name="inertia_origin_link_b">
         <origin xyz="5.1667E-06 0.069849 0.019496" rpy="0 0 0" />
 	</xacro:macro>
-	<xacro:macro name="origin_link_t">
+	<xacro:macro name="inertia_origin_link_t">
         <origin xyz="-0.00019051 0.0087466 -2.475E-05" rpy="0 0 0" />
 	</xacro:macro>
 	<xacro:macro name="default_joint_misc">
+		<!--
 		<calibration rising="0" falling="0"/>
 		<dynamics damping="0" fraction="0"/>
 		<safety_controller soft_upper="0" soft_lower="0" k_position="0" k_velocity="0"/>
+		-->
 	</xacro:macro>
 	<xacro:macro name="origin_joint_s">
@@ -69,9 +71,12 @@
         <origin xyz="0 0.164069662461231 0.0015" rpy="0 0 0" />
 	</xacro:macro>
+	<material name="white">
+		<color rgba="1 1 1 1"/>
+	</material>
 	<!-- base_link-->
 	<link name="base_link">
 		<inertial>
 			<mass value="1.0"/>
-			<xacro:default_origin/>
+			<xacro:inertia_origin_base_link/>
 			<xacro:default_mesh name="base_link"/>
 			<xacro:default_inertial/>
@@ -80,4 +85,5 @@
 			<xacro:default_origin/>
 			<xacro:default_mesh name="base_link"/>
+			<material name="white"/>
 		</visual>
 		<collision>
@@ -90,5 +96,5 @@
 		<inertial>
 			<mass value="1.0"/>
-			<xacro:default_origin/>
+			<xacro:inertia_origin_link_s/>
 			<xacro:default_mesh name="link_s"/>
 			<xacro:default_inertial/>
@@ -97,4 +103,5 @@
 			<xacro:default_origin/>
 			<xacro:default_mesh name="link_s"/>
+			<material name="white"/>
 		</visual>
 		<collision>
@@ -116,5 +123,5 @@
 		<inertial>
 			<mass value="1.0"/>
-			<xacro:default_origin/>
+			<xacro:inertia_origin_link_l/>
 			<xacro:default_mesh name="link_l"/>
 			<xacro:default_inertial/>
@@ -122,10 +129,9 @@
 		<visual>
 			<xacro:default_origin/>
-			<xacro:origin_link_l/>
 			<xacro:default_mesh name="link_l"/>
-		</visual>
-		<collision>
-			<xacro:default_origin/>
-			<xacro:origin_link_l/>
+			<material name="white"/>
+		</visual>
+		<collision>
+			<xacro:default_origin/>
 			<xacro:default_mesh name="link_l"/>
 		</collision>
@@ -144,5 +150,5 @@
 		<inertial>
 			<mass value="1.0"/>
-			<xacro:default_origin/>
+			<xacro:inertia_origin_link_e/>
 			<xacro:default_mesh name="link_e"/>
 			<xacro:default_inertial/>
@@ -151,4 +157,5 @@
 			<xacro:default_origin/>
 			<xacro:default_mesh name="link_e"/>
+			<material name="white"/>
 		</visual>
 		<collision>
@@ -170,5 +177,5 @@
 		<inertial>
 			<mass value="1.0"/>
-			<xacro:default_origin/>
+			<xacro:inertia_origin_link_u/>
 			<xacro:default_mesh name="link_u"/>
 			<xacro:default_inertial/>
@@ -177,8 +184,8 @@
 			<xacro:default_origin/>
 			<xacro:default_mesh name="link_u"/>
-		</visual>
-		<collision>
-			<xacro:default_origin/>
-			<xacro:default_mesh name="link_u"/>
+			<material name="white"/>
+		</visual>
+		<collision>
+			<xacro:default_origin/>
 			<xacro:default_mesh name="link_u"/>
 		</collision>
@@ -197,5 +204,5 @@
 		<inertial>
 			<mass value="1.0"/>
-			<xacro:default_origin/>
+			<xacro:inertia_origin_link_r/>
 			<xacro:default_mesh name="link_r"/>
 			<xacro:default_inertial/>
@@ -204,4 +211,5 @@
 			<xacro:default_origin/>
 			<xacro:default_mesh name="link_r"/>
+			<material name="white"/>
 		</visual>
 		<collision>
@@ -223,5 +231,5 @@
 		<inertial>
 			<mass value="1.0"/>
-			<xacro:default_origin/>
+			<xacro:inertia_origin_link_b/>
 			<xacro:default_mesh name="link_b"/>
 			<xacro:default_inertial/>
@@ -230,4 +238,5 @@
 			<xacro:default_origin/>
 			<xacro:default_mesh name="link_b"/>
+			<material name="white"/>
 		</visual>
 		<collision>
@@ -249,5 +258,5 @@
 		<inertial>
 			<mass value="1.0"/>
-			<xacro:default_origin/>
+			<xacro:inertia_origin_link_t/>
 			<xacro:default_mesh name="link_t"/>
 			<xacro:default_inertial/>
@@ -256,4 +265,5 @@
 			<xacro:default_origin/>
 			<xacro:default_mesh name="link_t"/>
+			<material name="white"/>
 		</visual>
 		<collision>
@@ -271,3 +281,27 @@
 		<xacro:default_joint_misc/>
 	</joint>
+	<!-- link tool0-->
+	<link name="tool0"/>
+	<!-- joint link_t-tool0 -->
+	<joint name="link_t-tool0" type="fixed">
+		<origin rpy="0 0 -3.1415" xyz="0 0 0"/>
+		<parent link="link_t"/>
+		<child  link="tool0"/>
+	</joint>
+	<!-- link fixed in order to stand rigidly in gazebo -->
+	<link name="world"/>
+	<joint name="fixed" type="fixed">
+		<orgin rpy="0 0 0" xyz="0 0 0"/>
+		<parent link="base_link"/>
+		<child  link="world"/>
+	</joint>
+	<!-- ros_control_plugin-->
+	<gazebo>
+		<plugin name="gazebo_ros_control" filename="libgazebo_ros_control.so">
+			<robotNamespace>/</robotNamespace>
+			<robotSimType>libgazebo_ros_control/DefaultRobotHWSim</robotSimType>
+		</plugin>
+		<mu1>0.3</mu1>
+		<mu2>0.3</mu2>
+	</gazebo>
 </robot>

File: urdf/sia20.urdf (robot description, URDF)
Before this commit: robot sia20, 8 links, 7 joints
Links:
- added link tool0
- added link world
- link base_link: mass 9.5604 -> 1.0; geometry collision mesh filename=package://sia20/meshes/base_link.STL; visual mesh filename=package://sia20/meshes/base_link.STL
- link link_b: mass 2.0184 -> 1.0; geometry collision mesh filename=package://sia20/meshes/link_b.STL; visual mesh filename=package://sia20/meshes/link_b.STL
- link link_e: mass 6.2419 -> 1.0; geometry collision mesh filename=package://sia20/meshes/link_e.STL; visual mesh filename=package://sia20/meshes/link_e.STL
- link link_l: mass 6.5581 -> 1.0; geometry collision mesh filename=package://sia20/meshes/link_l.STL; visual mesh filename=package://sia20/meshes/link_l.STL
- link link_r: mass 2.4173 -> 1.0; geometry collision mesh filename=package://sia20/meshes/link_r.STL; visual mesh filename=package://sia20/meshes/link_r.STL
- link link_s: mass 11.757 -> 1.0; geometry collision mesh filename=package://sia20/meshes/link_s.STL; visual mesh filename=package://sia20/meshes/link_s.STL
- link link_t: mass 0.095976 -> 1.0; geometry collision mesh filename=package://sia20/meshes/link_t.STL; visual mesh filename=package://sia20/meshes/link_t.STL
- link link_u: mass 4.4611 -> 1.0; geometry collision mesh filename=package://sia20/meshes/link_u.STL; visual mesh filename=package://sia20/meshes/link_u.STL
Joints:
- added joint fixed: type fixed, parent base_link, child world
- added joint link_t-tool0: type fixed, parent link_t, child tool0, origin xyz=0 0 0 rpy=0 0 -3.1415
- joint joint_b: type continuous -> revolute
- joint joint_e: limit lower=-2.9670 upper=2.9670 effort=100 velocity=2.9670 -> lower=-2.967 upper=2.967 effort=100 velocity=2.2698
- joint joint_l: limit lower=-1.9198 upper=1.9198 effort=100 velocity=2.2689 -> lower=-1.9198 upper=1.9198 effort=100 velocity=2.2698
- joint joint_r: limit lower=-3.1415 upper=3.1414 effort=100 velocity=3.4906 -> lower=-3.1415 upper=3.1415 effort=100 velocity=3.4906
- joint joint_s: limit lower=-3.1415 upper=3.1415 effort=100 velocity=2.2689 -> lower=-3.1415 upper=3.1415 effort=100 velocity=2.2698
- joint joint_t: limit lower=-3.14159 upper=3.14159 effort=100 velocity=7 -> lower=-3.1415 upper=3.1415 effort=100 velocity=7.0
- joint joint_u: limit lower=-2.9670 upper=2.9670 effort=100 velocity=2.9670 -> lower=-2.967 upper=2.967 effort=100 velocity=2.2698

Commit message: [update]

File: robots/sia20.urdf.xacro (robot description, xacro)
@@ -71,4 +71,16 @@
         <origin xyz="0 0.164069662461231 0.0015" rpy="0 0 0" />
 	</xacro:macro>
+	<xacro:macro name="default_transmission" params="suffix">
+		<transmission name="${suffix}_trans">
+			<type>transimission_interface/SimpleTransmission</type>
+			<joint name="${suffix}">
+				<hardwareInterface>hardware_interface/PositionJointInterface</hardwareInterface>
+			</joint>
+			<actuator name="${suffix}_motor">
+				<hardwareInterface>hardware_interface/PositionJointInterface</hardwareInterface>
+				<mechanicalReduction>1</mechanicalReduction>
+			</actuator>
+		</transmission>
+	</xacro:macro>
 	<material name="white">
 		<color rgba="1 1 1 1"/>
@@ -119,4 +131,5 @@
 		<xacro:default_joint_misc/>
 	</joint>
+	<xacro:default_transmission suffix="joint_s"/>
 	<!-- link_l-->
 	<link name="link_l">
@@ -146,4 +159,5 @@
 		<xacro:default_joint_misc/>
 	</joint>
+	<xacro:default_transmission suffix="joint_l"/>
 	<!-- link_e-->
 	<link name="link_e">
@@ -173,4 +187,5 @@
 		<xacro:default_joint_misc/>
 	</joint>
+	<xacro:default_transmission suffix="joint_e"/>
 	<!-- link_u-->
 	<link name="link_u">
@@ -200,4 +215,5 @@
 		<xacro:default_joint_misc/>
 	</joint>
+	<xacro:default_transmission suffix="joint_u"/>
 	<!-- link_r-->
 	<link name="link_r">
@@ -227,4 +243,5 @@
 		<xacro:default_joint_misc/>
 	</joint>
+	<xacro:default_transmission suffix="joint_r"/>
 	<!-- link_b-->
 	<link name="link_b">
@@ -254,4 +271,5 @@
 		<xacro:default_joint_misc/>
 	</joint>
+	<xacro:default_transmission suffix="joint_b"/>
 	<!-- link_t-->
 	<link name="link_t">
@@ -281,4 +299,5 @@
 		<xacro:default_joint_misc/>
 	</joint>
+	<xacro:default_transmission suffix="joint_t"/>
 	<!-- link tool0-->
 	<link name="tool0"/>
@@ -292,16 +311,14 @@
 	<link name="world"/>
 	<joint name="fixed" type="fixed">
-		<orgin rpy="0 0 0" xyz="0 0 0"/>
-		<parent link="base_link"/>
-		<child  link="world"/>
+		<parent link="world"/>
+		<child  link="base_link"/>
 	</joint>
 	<!-- ros_control_plugin-->
 	<gazebo>
 		<plugin name="gazebo_ros_control" filename="libgazebo_ros_control.so">
-			<robotNamespace>/</robotNamespace>
-			<robotSimType>libgazebo_ros_control/DefaultRobotHWSim</robotSimType>
+			<robotNameSpace>/sia20</robotNameSpace>
 		</plugin>
-		<mu1>0.3</mu1>
-		<mu2>0.3</mu2>
+		<mu1>0.1</mu1>
+		<mu2>0.1</mu2>
 	</gazebo>
 </robot>

File: urdf/sia20.urdf (robot description, URDF)
Before this commit: robot sia20, 10 links, 9 joints
Joints:
- joint fixed: child world -> base_link; parent base_link -> world
