Commit message: [add] added sia20_control and readme.md

File: sia20_description/robots/sia20.urdf.xacro (robot description, xacro)
@@ -4,5 +4,5 @@
 	<xacro:macro name="default_mesh" params="name">
 		<geometry>
-			<mesh filename="package://sia20/meshes/${name}.STL"/>
+			<mesh filename="package://sia20_description/meshes/${name}.STL"/>
 		</geometry>
 	</xacro:macro>
@@ -317,5 +317,5 @@
 	<gazebo>
 		<plugin name="gazebo_ros_control" filename="libgazebo_ros_control.so">
-			<robotNamespace>/</robotNamespace>
+			<robotNamespace>/sia20</robotNamespace>
 		</plugin>
 		<mu1>0.1</mu1>
