Commit message: [add] added sia20_with_gripper.urdf.xacro

File: sia20_description/robots/gripper.urdf.xacro (robot description, xacro)
@@ -1,4 +1,46 @@
 <?xml version="1.0"?>
-<robot name="sia20" xmlns:xacro="http://ros.org/wiki/xacro">
-<!-- copied from line 159 11-gripper.urdf.xacro-->
-<!-- right gripper and left one exist, therfore, macro is made -->
+<robot name="sia20" xmlns:xacro="http://www.ros.org/wiki/xacro">
+	<!-- copied from line 159 11-gripper.urdf.xacro-->
+	<!-- right gripper and left one exist, therfore, macro is made -->
+	<xacro:macro name="gripper" params="prefix">
+		<link name="${prefix}_gripper">
+			<inertial>
+				<xacro:default_origin/>
+				<geometory>
+					<mash filename="package://urdf_tutorial/meshes/l_finger.dae"/>
+				</geometory>
+				<xacro:default_inertial/>
+				<mass value="0.01"/>
+			</inertial>
+			<visual>
+				<origin rpy="0 0 0" xyz="0 0 0"/>
+				<geometory>
+					<mash filename="package://urdf_tutorial/meshes/l_finger.dae"/>
+				</geometory>
+			</visual>
+			<collision>
+				<origin rpy="0 0 0" xyz="0 0 0"/>
+				<geometory>
+					<mash filename="package://urdf_tutorial/meshes/l_finger.dae"/>
+				</geometory>
+			</collision>
+		</link>
+		<joint name="${prefix}_gripper_joint" type="revolute">
+			<axis xyz="0 0 0"/>
+			<origin rpy="0 0 0" xyz="0 0 0"/>
+			<limit effort="1000" lower="0.0" upper="0.548" velocity="1"/>
+			<parent link="tool0"/>
+			<child  link="${prefix}_gripper"/>
+		</joint>
+		<transmission name="${prefix}_gripper_trans" type="SimpleTransmission">
+			<type>transmission_interface/SimpleTransmission</type>
+			<actuator name="${prefix}_gripper_motor">
+				<mechanicalReduction>1</mechanicalReduction>
+				<hardwareInterface>PositionJointInterface</hardwareInterface>
+			</actuator>
+			<joint name="${prefix}_gripper_joint">
+				<hardwareInterface>PositionJointInterface</hardwareInterface>
+			</joint>
+		</transmission>
+	</xacro:macro>
+</robot>

Commit message: [update] only visual, complete gripper xacro and attached to robot

File: sia20_description/robots/gripper.urdf.xacro (robot description, xacro)
@@ -1,46 +1,41 @@
 <?xml version="1.0"?>
 <robot name="sia20" xmlns:xacro="http://www.ros.org/wiki/xacro">
-	<!-- copied from line 159 11-gripper.urdf.xacro-->
-	<!-- right gripper and left one exist, therfore, macro is made -->
-	<xacro:macro name="gripper" params="prefix">
-		<link name="${prefix}_gripper">
-			<inertial>
-				<xacro:default_origin/>
-				<geometory>
-					<mash filename="package://urdf_tutorial/meshes/l_finger.dae"/>
-				</geometory>
-				<xacro:default_inertial/>
-				<mass value="0.01"/>
-			</inertial>
-			<visual>
-				<origin rpy="0 0 0" xyz="0 0 0"/>
-				<geometory>
-					<mash filename="package://urdf_tutorial/meshes/l_finger.dae"/>
-				</geometory>
-			</visual>
-			<collision>
-				<origin rpy="0 0 0" xyz="0 0 0"/>
-				<geometory>
-					<mash filename="package://urdf_tutorial/meshes/l_finger.dae"/>
-				</geometory>
-			</collision>
-		</link>
-		<joint name="${prefix}_gripper_joint" type="revolute">
-			<axis xyz="0 0 0"/>
-			<origin rpy="0 0 0" xyz="0 0 0"/>
-			<limit effort="1000" lower="0.0" upper="0.548" velocity="1"/>
-			<parent link="tool0"/>
-			<child  link="${prefix}_gripper"/>
-		</joint>
-		<transmission name="${prefix}_gripper_trans" type="SimpleTransmission">
-			<type>transmission_interface/SimpleTransmission</type>
-			<actuator name="${prefix}_gripper_motor">
-				<mechanicalReduction>1</mechanicalReduction>
-				<hardwareInterface>PositionJointInterface</hardwareInterface>
-			</actuator>
-			<joint name="${prefix}_gripper_joint">
-				<hardwareInterface>PositionJointInterface</hardwareInterface>
-			</joint>
-		</transmission>
-	</xacro:macro>
+	<!-- include common macro file-->
+	<xacro:include filename="common.urdf.xacro" />
+	<link name="left_gripper">
+		<collision>
+			<origin rpy="0 0 -1.5708" xyz="0.01 -0.02 0"/>
+			<geometry>
+				<mesh filename="package://urdf_tutorial/meshes/l_finger.dae"/>
+			</geometry>
+		</collision>
+		<inertial>
+			<mass value="0.01"/>
+			<xacro:default_inertial/>
+		</inertial>
+		<visual>
+			<origin rpy="0 0 -1.5708" xyz="0.01 -0.02 0"/>
+			<geometry>
+				<mesh filename="package://urdf_tutorial/meshes/l_finger.dae"/>
+			</geometry>
+		</visual>
+	</link>
+	<link name="right_gripper">
+		<collision>
+			<origin rpy="3.14 0 -1.5708" xyz="-0.01 -0.02 0"/>
+			<geometry>
+				<mesh filename="package://urdf_tutorial/meshes/l_finger.dae"/>
+			</geometry>
+		</collision>
+		<inertial>
+			<mass value="0.01"/>
+			<xacro:default_inertial/>
+		</inertial>
+		<visual>
+			<origin rpy="3.14 0 -1.5708" xyz="-0.01 -0.02 0"/>
+			<geometry>
+				<mesh filename="package://urdf_tutorial/meshes/l_finger.dae"/>
+			</geometry>
+		</visual>
+	</link>
 </robot>

File: sia20_description/robots/sia20.urdf.xacro (robot description, xacro)
@@ -1,89 +1,6 @@
 <?xml version="1.0"?>
 <robot name="sia20" xmlns:xacro="http://www.ros.org/wiki/xacro">
-	<!-- macro -->
-	<xacro:macro name="default_mesh" params="name">
-		<geometry>
-			<mesh filename="package://sia20_description/meshes/${name}.STL"/>
-		</geometry>
-	</xacro:macro>
-	<xacro:macro name="default_inertial">
-		<inertia
-			ixx="0.001"
-			ixy="0.001"
-			ixz="0.001"
-			iyy="0.001"
-			iyz="0.001"
-			izz="0.001"/>
-	</xacro:macro>
-	<xacro:macro name="default_origin">
-		<origin xyz="0 0 0" rpy="0 0 0" />
-	</xacro:macro>
-	<xacro:macro name="inertia_origin_base_link">
-		<origin xyz="-0.05327 0.066798 0.00014271" rpy="0 0 0" />
-	</xacro:macro>
-	<xacro:macro name="inertia_origin_link_s">
-        <origin xyz="7.8023E-07 0.18911 -0.015611" rpy="0 0 0" />
-	</xacro:macro>
-	<xacro:macro name="inertia_origin_link_l">
-        <origin xyz="1.6057E-05 0.10201 0.041335" rpy="0 0 0" />
-	</xacro:macro>
-	<xacro:macro name="inertia_origin_link_e">
-        <origin xyz="3.9186E-05 0.16471 0.020774" rpy="0 0 0" />
-	</xacro:macro>
-	<xacro:macro name="inertia_origin_link_u">
-        <origin xyz="-7.9992E-07 0.08472 -0.032542" rpy="0 0 0" />
-	</xacro:macro>
-	<xacro:macro name="inertia_origin_link_r">
-        <origin xyz="4.8678E-06 0.12569 -0.02028" rpy="0 0 0" />
-	</xacro:macro>
-	<xacro:macro name="inertia_origin_link_b">
-        <origin xyz="5.1667E-06 0.069849 0.019496" rpy="0 0 0" />
-	</xacro:macro>
-	<xacro:macro name="inertia_origin_link_t">
-        <origin xyz="-0.00019051 0.0087466 -2.475E-05" rpy="0 0 0" />
-	</xacro:macro>
-	<xacro:macro name="default_joint_misc">
-		<!--
-		<calibration rising="0" falling="0"/>
-		<dynamics damping="0" fraction="0"/>
-		<safety_controller soft_upper="0" soft_lower="0" k_position="0" k_velocity="0"/>
-		-->
-	</xacro:macro>
-	<xacro:macro name="origin_joint_s">
-        <origin xyz="0 0 0.112" rpy="1.5708 0 0" />
-	</xacro:macro>
-	<xacro:macro name="origin_joint_l">
-        <origin xyz="0 0.298 0" rpy="0 0 0" />
-	</xacro:macro>
-	<xacro:macro name="origin_joint_e">
-        <origin xyz="0 0.247135547651375 0" rpy="0 0 0" />
-	</xacro:macro>
-	<xacro:macro name="origin_joint_u">
-        <origin xyz="0 0.242864452348634 0" rpy="0 0 0" />
-	</xacro:macro>
-	<xacro:macro name="origin_joint_r">
-        <origin xyz="0 0.23899999999989 0" rpy="0 0 0" />
-	</xacro:macro>
-	<xacro:macro name="origin_joint_b">
-        <origin xyz="0 0.181 0" rpy="0 0 0" />
-	</xacro:macro>
-	<xacro:macro name="origin_joint_t">
-        <origin xyz="0 0.164069662461231 0.0015" rpy="0 0 0" />
-	</xacro:macro>
-	<xacro:macro name="default_transmission" params="suffix">
-		<transmission name="${suffix}_trans">
-			<type>transimission_interface/SimpleTransmission</type>
-			<joint name="${suffix}">
-				<hardwareInterface>hardware_interface/EffortJointInterface</hardwareInterface>
-			</joint>
-			<actuator name="${suffix}_motor">
-				<hardwareInterface>hardware_interface/EffortJointInterface</hardwareInterface>
-				<mechanicalReduction>1</mechanicalReduction>
-			</actuator>
-		</transmission>
-	</xacro:macro>
-	<material name="white">
-		<color rgba="1 1 1 1"/>
-	</material>
+	<!-- include macro file-->
+	<xacro:include filename="common.urdf.xacro"/>
 	<!-- base_link-->
 	<link name="base_link">

File: sia20_description/robots/sia20_with_gripper.urdf.xacro (robot description, xacro)
@@ -2,8 +2,15 @@
 <robot name="sia20" xmlns:xacro="http://www.ros.org/wiki/xacro">
 	<!-- include robot -->
-	<xacro:include filename="$(find sia20_description)/robots/sia20.urdf.xacro" />
+	<xacro:include filename="sia20.urdf.xacro" />
 	<!-- include gripper -->
-	<xacro:include filename="$(find sia20_description)/robots/gripper.urdf.xacro" />
+	<xacro:include filename="gripper.urdf.xacro" />
 	<!-- concatenate gripper to robot -->
-	<xacro:gripper prefix="left" />
+	<joint name="wrist_to_l" type="fixed">
+		<parent  link="tool0"/>
+		<child link="left_gripper"/>
+	</joint>
+	<joint name="wrist_to_r" type="fixed">
+		<parent link="tool0"/>
+		<child link="right_gripper"/>
+	</joint>
 </robot>

Commit message: [update] added gripper urdf and config and launch file. but not work

File: sia20_description/robots/gripper.urdf.xacro (robot description, xacro)
@@ -5,5 +5,5 @@
 	<link name="left_gripper">
 		<collision>
-			<origin rpy="0 0 -1.5708" xyz="0.01 -0.02 0"/>
+			<origin rpy="0 0 -1.5708" xyz="0.013 -0.02 0"/>
 			<geometry>
 				<mesh filename="package://urdf_tutorial/meshes/l_finger.dae"/>
@@ -15,5 +15,5 @@
 		</inertial>
 		<visual>
-			<origin rpy="0 0 -1.5708" xyz="0.01 -0.02 0"/>
+			<origin rpy="0 0 -1.5708" xyz="0.013 -0.02 0"/>
 			<geometry>
 				<mesh filename="package://urdf_tutorial/meshes/l_finger.dae"/>
@@ -23,5 +23,5 @@
 	<link name="right_gripper">
 		<collision>
-			<origin rpy="3.14 0 -1.5708" xyz="-0.01 -0.02 0"/>
+			<origin rpy="3.14 0 -1.5708" xyz="-0.013 -0.02 0"/>
 			<geometry>
 				<mesh filename="package://urdf_tutorial/meshes/l_finger.dae"/>
@@ -33,5 +33,5 @@
 		</inertial>
 		<visual>
-			<origin rpy="3.14 0 -1.5708" xyz="-0.01 -0.02 0"/>
+			<origin rpy="3.14 0 -1.5708" xyz="-0.013 -0.02 0"/>
 			<geometry>
 				<mesh filename="package://urdf_tutorial/meshes/l_finger.dae"/>

File: sia20_description/robots/sia20_with_gripper.urdf.xacro (robot description, xacro)
@@ -6,11 +6,43 @@
 	<xacro:include filename="gripper.urdf.xacro" />
 	<!-- concatenate gripper to robot -->
-	<joint name="wrist_to_l" type="fixed">
+	<joint name="wrist_to_l" type="revolute">
 		<parent  link="tool0"/>
 		<child link="left_gripper"/>
+		<limit effort="1000" lower="-0.07" upper="0.548" velocity="3"/>
+		<axis xyz="0 0 1"/>
 	</joint>
-	<joint name="wrist_to_r" type="fixed">
+	<joint name="wrist_to_r" type="revolute">
 		<parent link="tool0"/>
 		<child link="right_gripper"/>
+		<limit effort="1000" lower="-0.07" upper="0.548" velocity="3"/>
+		<axis xyz="0 0 -1"/>
 	</joint>
+	<!-- transmission -->
+	<transmission name="left_gripper_trans">
+		<type>transmission_interface/SimpleTransmission</type>
+		<joint name="wrist_to_l">
+			<hardwareInterface>hardware_interface/EffortJointInterface</hardwareInterface>
+		</joint>
+		<actuator name="wrist_to_l_motor">
+			<hardwareInterface>hardware_interface/EffortJointInterface</hardwareInterface>
+			<mechanicalReduction>1</mechanicalReduction>
+		</actuator>
+	</transmission>
+	<transmission name="right_gripper_trans">
+		<type>transmission_interface/SimpleTransmission</type>
+		<joint name="wrist_to_r">
+			<hardwareInterface>hardware_interface/EffortJointInterface</hardwareInterface>
+		</joint>
+		<actuator name="wrist_to_r_motor">
+			<hardwareInterface>hardware_interface/EffortJointInterface</hardwareInterface>
+			<mechanicalReduction>1</mechanicalReduction>
+		</actuator>
+	</transmission>
+	<gazebo>
+		<plugin name="gazebo_ros_control" filename="libgazebo_ros_control.so">
+			<robotNamespace>/sia20</robotNamespace>
+		</plugin>
+		<mu1>0.1</mu1>
+		<mu2>0.1</mu2>
+	</gazebo>
 </robot>

Commit message: [update] add gripper tip

File: sia20_description/robots/gripper.urdf.xacro (robot description, xacro)
@@ -21,15 +21,27 @@
 		</visual>
 	</link>
-	<link name="right_gripper">
+	<link name="left_tip">
+		<visual>
+			<origin rpy="0 0 0" xyz="0.09137 0.00495 0"/>
+			<geometry>
+				<mesh filename="package://urdf_tutorial/meshes/l_finger_tip.dae"/>
+			</geometry>
+		</visual>
 		<collision>
-			<origin rpy="3.14 0 -1.5708" xyz="-0.013 -0.02 0"/>
 			<geometry>
-				<mesh filename="package://urdf_tutorial/meshes/l_finger.dae"/>
+				<mesh filename="package://urdf_tutorial/meshes/l_finger_tip.dae"/>
 			</geometry>
+			<origin rpy="0 0 0" xyz="0.09137 0.00495 0"/>
 		</collision>
 		<inertial>
 			<mass value="0.01"/>
-			<xacro:default_inertial/>
+			<inertia ixx="0.1" ixy="0.1" ixz="0.1" iyy="0.1" iyz="0.1" izz="0.1"/>
 		</inertial>
+	</link>
+	<joint name="left_tip_joint" type="fixed">
+		<parent link="left_gripper"/>
+		<child  link="left_tip"/>
+	</joint>
+	<link name="right_gripper">
 		<visual>
 			<origin rpy="3.14 0 -1.5708" xyz="-0.013 -0.02 0"/>
@@ -38,4 +50,36 @@
 			</geometry>
 		</visual>
+		<collision>
+			<geometry>
+				<mesh filename="package://urdf_tutorial/meshes/l_finger.dae"/>
+			</geometry>
+			<origin rpy="3.14 0 -1.5708" xyz="-0.013 -0.02 0"/>
+		</collision>
+		<inertial>
+			<mass value="0.01"/>
+			<xacro:default_inertial/>
+		</inertial>
 	</link>
+	<link name="right_tip">
+		<visual>
+			<origin rpy="3.14 0 0" xyz="0.09137 0.00495 0"/>
+			<geometry>
+				<mesh filename="package://urdf_tutorial/meshes/l_finger_tip.dae"/>
+			</geometry>
+		</visual>
+		<collision>
+			<geometry>
+				<mesh filename="package://urdf_tutorial/meshes/l_finger_tip.dae"/>
+			</geometry>
+			<origin rpy="3.14 0 0" xyz="0.09137 0.00495 0"/>
+		</collision>
+		<inertial>
+			<mass value="0.01"/>
+			<inertia ixx="0.1" ixy="0.1" ixz="0.1" iyy="0.1" iyz="0.1" izz="0.1"/>
+		</inertial>
+	</link>
+	<joint name="right_tip_joint" type="fixed">
+		<parent link="right_gripper"/>
+		<child  link="right_tip"/>
+	</joint>
 </robot>

File: sia20_description/robots/model.urdf (robot description, URDF)
Before this commit: robot sia20, 12 links, 11 joints
Links:
- added link left_tip, mass 0.01; collision mesh filename=package://urdf_tutorial/meshes/l_finger_tip.dae; visual mesh filename=package://urdf_tutorial/meshes/l_finger_tip.dae
- added link right_tip, mass 0.01; collision mesh filename=package://urdf_tutorial/meshes/l_finger_tip.dae; visual mesh filename=package://urdf_tutorial/meshes/l_finger_tip.dae
- link right_gripper: geometry collision mesh filename=package://urdf_tutorial/meshes/l_finger.dae; visual mesh filename=package://urdf_tutorial/meshes/l_finger.dae
Joints:
- added joint left_tip_joint: type fixed, parent left_gripper, child left_tip
- joint wrist_to_l: axis (none) -> 0 0 1; limit (none) -> lower=-0.07 upper=0.548 effort=1000 velocity=3; type fixed -> revolute
- joint wrist_to_r: axis (none) -> 0 0 -1; limit (none) -> lower=-0.07 upper=0.548 effort=1000 velocity=3; type fixed -> revolute

Commit message: [update] getting error : This robot has a joint named foo which is not in the gazebo model.

File: sia20_description/robots/gripper.urdf.xacro (robot description, xacro)
@@ -12,5 +12,5 @@
 		<inertial>
 			<mass value="0.01"/>
-			<xacro:default_inertial/>
+			<inertia ixx="0.1" ixy="0.1" ixz="0.1" iyy="0.1" iyz="0.1" izz="0.1"/>
 		</inertial>
 		<visual>
@@ -58,5 +58,5 @@
 		<inertial>
 			<mass value="0.01"/>
-			<xacro:default_inertial/>
+			<inertia ixx="0.1" ixy="0.1" ixz="0.1" iyy="0.1" iyz="0.1" izz="0.1"/>
 		</inertial>
 	</link>

File: sia20_description/robots/model.urdf (robot description, URDF)
Before this commit: robot sia20, 14 links, 12 joints
Joints:
- added joint right_tip_joint: type fixed, parent right_gripper, child right_tip
- joint wrist_to_l: parent tool0 -> link_t
- joint wrist_to_r: parent tool0 -> link_t

File: sia20_description/robots/sia20_with_gripper.urdf.xacro (robot description, xacro)
@@ -7,12 +7,12 @@
 	<!-- concatenate gripper to robot -->
 	<joint name="wrist_to_l" type="revolute">
-		<parent  link="tool0"/>
-		<child link="left_gripper"/>
+		<parent  link="link_t"/>
+		<child   link="left_gripper"/>
 		<limit effort="1000" lower="-0.07" upper="0.548" velocity="3"/>
 		<axis xyz="0 0 1"/>
 	</joint>
 	<joint name="wrist_to_r" type="revolute">
-		<parent link="tool0"/>
-		<child link="right_gripper"/>
+		<parent  link="link_t"/>
+		<child   link="right_gripper"/>
 		<limit effort="1000" lower="-0.07" upper="0.548" velocity="3"/>
 		<axis xyz="0 0 -1"/>

Commit message: [update] error fixing now

File: sia20_description/robots/gripper.urdf.xacro (robot description, xacro)
@@ -5,5 +5,5 @@
 	<link name="left_gripper">
 		<collision>
-			<origin rpy="0 0 -1.5708" xyz="0.013 -0.02 0"/>
+			<origin rpy="0 0 0" xyz="0 0 0"/>
 			<geometry>
 				<mesh filename="package://urdf_tutorial/meshes/l_finger.dae"/>
@@ -15,5 +15,5 @@
 		</inertial>
 		<visual>
-			<origin rpy="0 0 -1.5708" xyz="0.013 -0.02 0"/>
+			<origin rpy="0 0 0" xyz="0 0 0"/>
 			<geometry>
 				<mesh filename="package://urdf_tutorial/meshes/l_finger.dae"/>
@@ -45,5 +45,5 @@
 	<link name="right_gripper">
 		<visual>
-			<origin rpy="3.14 0 -1.5708" xyz="-0.013 -0.02 0"/>
+			<origin rpy="0 0 0" xyz="-0.013 -0.02 0"/>
 			<geometry>
 				<mesh filename="package://urdf_tutorial/meshes/l_finger.dae"/>
@@ -54,5 +54,5 @@
 				<mesh filename="package://urdf_tutorial/meshes/l_finger.dae"/>
 			</geometry>
-			<origin rpy="3.14 0 -1.5708" xyz="-0.013 -0.02 0"/>
+			<origin rpy="0 0 0" xyz="-0.013 -0.02 0"/>
 		</collision>
 		<inertial>

File: sia20_description/robots/sia20_with_gripper.urdf.xacro (robot description, xacro)
@@ -10,4 +10,5 @@
 		<child   link="left_gripper"/>
 		<limit effort="1000" lower="-0.07" upper="0.548" velocity="3"/>
+		<origin rpy="0 0 0" xyz="0.2 0.01 0"/>
 		<axis xyz="0 0 1"/>
 	</joint>
@@ -16,4 +17,5 @@
 		<child   link="right_gripper"/>
 		<limit effort="1000" lower="-0.07" upper="0.548" velocity="3"/>
+		<origin rpy="0 0 0" xyz="0.2 -0.01 0"/>
 		<axis xyz="0 0 -1"/>
 	</joint>

Commit message: [update] gripper is complete for now

File: sia20_description/robots/gripper.urdf.xacro (robot description, xacro)
@@ -45,5 +45,5 @@
 	<link name="right_gripper">
 		<visual>
-			<origin rpy="0 0 0" xyz="-0.013 -0.02 0"/>
+			<origin rpy="3.14 0 0" xyz="0 0 0"/>
 			<geometry>
 				<mesh filename="package://urdf_tutorial/meshes/l_finger.dae"/>
@@ -54,5 +54,5 @@
 				<mesh filename="package://urdf_tutorial/meshes/l_finger.dae"/>
 			</geometry>
-			<origin rpy="0 0 0" xyz="-0.013 -0.02 0"/>
+			<origin rpy="3.14 0 0" xyz="0 0 0"/>
 		</collision>
 		<inertial>
