Commit message: [update] aligned gripper's gap and length between grippers and arm

File: sia20_description/robots/sia20_with_gripper.urdf.xacro (robot description, xacro)
@@ -9,6 +9,7 @@
 		<parent  link="link_t"/>
 		<child   link="left_gripper"/>
-		<limit effort="1000" lower="-0.07" upper="0.548" velocity="3"/>
-		<origin rpy="0 0 0" xyz="0.2 0.01 0"/>
+		<limit effort="1000" lower="0" upper="0.548" velocity="3"/>
+		<!-- In order to expand the width between two grippers, change x value -->
+		<origin rpy="0 0 1.5708" xyz="-0.01 0.04 0"/>
 		<axis xyz="0 0 1"/>
 	</joint>
@@ -16,6 +17,7 @@
 		<parent  link="link_t"/>
 		<child   link="right_gripper"/>
-		<limit effort="1000" lower="-0.07" upper="0.548" velocity="3"/>
-		<origin rpy="0 0 0" xyz="0.2 -0.01 0"/>
+		<limit effort="1000" lower="0" upper="0.548" velocity="3"/>
+		<!-- In order to expand the width between two grippers, change x value -->
+		<origin rpy="0 0 1.5708" xyz="0.01 0.04 0"/>
 		<axis xyz="0 0 -1"/>
 	</joint>
