Commit message: [update] recovered color tag in sia20.urdf.xacro

File: sia20_description/robots/common.urdf.xacro (robot description, xacro)
@@ -1,4 +1,8 @@
 <?xml version="1.0"?>
 <robot name="sia20" xmlns:xacro="http://www.ros.org/wiki/xacro">
+	<!-- color of robot. important-->
+	<material name="white">
+		<color rgba="1 1 1 1"/>
+	</material>
 	<!-- Defitnitions of convinience macro -->
 	<xacro:macro name="default_mesh" params="name">

Commit message: [update] set sim env

File: sia20_description/robots/common.urdf.xacro (robot description, xacro)
@@ -79,8 +79,8 @@
 			<type>transimission_interface/SimpleTransmission</type>
 			<joint name="${suffix}">
-				<hardwareInterface>hardware_interface/EffortJointInterface</hardwareInterface>
+				<hardwareInterface>hardware_interface/PositionJointInterface</hardwareInterface>
 			</joint>
 			<actuator name="${suffix}_motor">
-				<hardwareInterface>hardware_interface/EffortJointInterface</hardwareInterface>
+				<hardwareInterface>hardware_interface/PositionJointInterface</hardwareInterface>
 				<mechanicalReduction>1</mechanicalReduction>
 			</actuator>

File: sia20_description/robots/sia20.urdf.xacro (robot description, xacro)
@@ -46,5 +46,5 @@
 		<child  link="link_s"/>
 		<axis xyz="0 1 0"/>
-		<limit lower="-3.1415" upper="3.1415" effort="100" velocity="2.2698"/>
+		<limit lower="-3.1415" upper="3.1415" effort="1000" velocity="2.2698"/>
 		<xacro:default_joint_misc/>
 	</joint>
@@ -74,5 +74,5 @@
 		<child  link="link_l"/>
 		<axis xyz="0 0 1"/>
-		<limit lower="-1.9198" upper="1.9198" effort="100" velocity="2.2698"/>
+		<limit lower="-1.9198" upper="1.9198" effort="1000" velocity="2.2698"/>
 		<xacro:default_joint_misc/>
 	</joint>
@@ -102,5 +102,5 @@
 		<child  link="link_e"/>
 		<axis xyz="0 1 0"/>
-		<limit lower="-2.967" upper="2.967" effort="100" velocity="2.2698"/>
+		<limit lower="-2.967" upper="2.967" effort="1000" velocity="2.2698"/>
 		<xacro:default_joint_misc/>
 	</joint>
@@ -130,5 +130,5 @@
 		<child  link="link_u"/>
 		<axis xyz="0 0 1"/>
-		<limit lower="-2.967" upper="2.967" effort="100" velocity="2.2698"/>
+		<limit lower="-2.967" upper="2.967" effort="1000" velocity="2.2698"/>
 		<xacro:default_joint_misc/>
 	</joint>
@@ -158,5 +158,5 @@
 		<child  link="link_r"/>
 		<axis xyz="0 1 0"/>
-		<limit lower="-3.1415" upper="3.1415" effort="100" velocity="3.4906"/>
+		<limit lower="-3.1415" upper="3.1415" effort="1000" velocity="3.4906"/>
 		<xacro:default_joint_misc/>
 	</joint>
@@ -186,5 +186,5 @@
 		<child  link="link_b"/>
 		<axis xyz="0 0 1"/>
-		<limit lower="-1.9198" upper="1.9198" effort="100" velocity="3.4906"/>
+		<limit lower="-1.9198" upper="1.9198" effort="1000" velocity="3.4906"/>
 		<xacro:default_joint_misc/>
 	</joint>
@@ -214,5 +214,5 @@
 		<child  link="link_t"/>
 		<axis xyz="0 1 0"/>
-		<limit lower="-3.1415" upper="3.1415" effort="100" velocity="7.0"/>
+		<limit lower="-3.1415" upper="3.1415" effort="1000" velocity="7.0"/>
 		<xacro:default_joint_misc/>
 	</joint>
