Commit message: [update] clean up sia20_description/launch

File: sia20_description/urdf/sia20.urdf (robot description, URDF)
Before this commit: robot sia20, 10 links, 9 joints
Links:
- link base_link: geometry collision mesh filename=package://sia20_description/meshes/base_link.STL; visual mesh filename=package://sia20_description/meshes/base_link.STL
- link link_b: geometry collision mesh filename=package://sia20_description/meshes/link_b.STL; visual mesh filename=package://sia20_description/meshes/link_b.STL
- link link_e: geometry collision mesh filename=package://sia20_description/meshes/link_e.STL; visual mesh filename=package://sia20_description/meshes/link_e.STL
- link link_l: geometry collision mesh filename=package://sia20_description/meshes/link_l.STL; visual mesh filename=package://sia20_description/meshes/link_l.STL
- link link_r: geometry collision mesh filename=package://sia20_description/meshes/link_r.STL; visual mesh filename=package://sia20_description/meshes/link_r.STL
- link link_s: geometry collision mesh filename=package://sia20_description/meshes/link_s.STL; visual mesh filename=package://sia20_description/meshes/link_s.STL
- link link_t: geometry collision mesh filename=package://sia20_description/meshes/link_t.STL; visual mesh filename=package://sia20_description/meshes/link_t.STL
- link link_u: geometry collision mesh filename=package://sia20_description/meshes/link_u.STL; visual mesh filename=package://sia20_description/meshes/link_u.STL
