Commit message: [update] for now. Spawn only broom in gazebo

File: sia20_gazebo/urdf/broom.urdf (robot description, URDF)
Before this commit: robot broom, 2 links, 1 joints
Links:
- link broom_foot: geometry collision mesh filename=package://broom/broom_foot.STL; visual mesh filename=package://broom/broom_foot.STL
- link broom_head: geometry collision mesh filename=package://broom/broom_head.STL; visual mesh filename=package://broom/broom_head.STL

Commit message: [update] in sia20_gazebo package, all sim enviroment complete

File: sia20_gazebo/urdf/broom.urdf (robot description, URDF)
Before this commit: robot broom, 2 links, 1 joints
Links:
- link broom_foot: mass 0.27406 -> 0.3; geometry collision mesh filename=package://broom/meshes/broom_foot.STL; visual mesh filename=package://broom/meshes/broom_foot.STL
- link broom_head: mass 0.15357 -> 0.3; geometry collision mesh filename=package://broom/meshes/broom_head.STL; visual mesh filename=package://broom/meshes/broom_head.STL
Joints:
- joint broom_joint: limit lower=-0.785 upper=785 effort=0 velocity=0 -> lower=-0.785 upper=0.785 effort=0 velocity=0
